Commit message: thrusters are pretty close to centered

File: urdf/robots/brov2_description/urdf/brov2.gazebo.xacro (robot description, xacro)
@@ -16,5 +16,5 @@
     Center of buoyancy according to Table 5.1 p. 48 in Wu2018.
     -->
-    <xacro:property name="cob" value="0.0 0.0 0.2"/>
+    <xacro:property name="cob" value="0.0 0.0 0.0"/>
     <!-- overestimated cube based on brov2 dimensions https://bluerobotics.com/store/rov/bluerov2-upgrade-kits/brov2-heavy-retrofit/ -->
     <xacro:property name="volume" value="0.0661"/>
@@ -40,9 +40,9 @@
                     0.0   0.0  0.0     0.0   0.0  -0.12
                 </added_mass>
-                <!-- Linear Damping: see p.28 Table 5.3 p. 48 in Wu2018 -->
+                <!-- Linear Damping: see Table 5.3 p. 48 in Wu2018 -->
                 <linear_damping>
                     -4.03 -6.22 -5.18 -0.07 -0.07 -0.07
                 </linear_damping>
-                <!-- Non-linear Damping: see p.28 Table 5.3 p. 48 in Wu2018 -->
+                <!-- Non-linear Damping: see Table 5.3 p. 48 in Wu2018 -->
                 <quadratic_damping>
                     -18.18 -21.66 -36.99 -1.55 -1.55 -1.55
@@ -51,3 +51,11 @@
         </link>
     </xacro:macro>
+                <!-- <added_mass>
+                    5.5   0.0  0.0    0.0   0.0   0.0
+                    0.0   12.7 0.0    0.0   0.0   0.0
+                    0.0   0.0  14.57  0.0   0.0   0.0
+                    0.0   0.0  0.0    0.12  0.0   0.0
+                    0.0   0.0  0.0    0.0   0.12  0.0
+                    0.0   0.0  0.0    0.0   0.0   0.12
+                </added_mass> -->
 </robot>

Commit message: thrusters are pretty close to centered

File: urdf/robots/brov2_description/urdf/brov2.gazebo.xacro (robot description, xacro)
@@ -16,5 +16,5 @@
     Center of buoyancy according to Table 5.1 p. 48 in Wu2018.
     -->
-    <xacro:property name="cob" value="0.0 0.0 0.2"/>
+    <xacro:property name="cob" value="0.0 0.0 0.0"/>
     <!-- overestimated cube based on brov2 dimensions https://bluerobotics.com/store/rov/bluerov2-upgrade-kits/brov2-heavy-retrofit/ -->
     <xacro:property name="volume" value="0.0661"/>

File: urdf/robots/brov2_description/urdf/brov2_actuators.xacro (robot description, xacro)
@@ -13,5 +13,5 @@
 -->
 <robot xmlns:xacro="http://www.ros.org/wiki/xacro">
-  <xacro:property name="prop_mesh_file" value="file://$(find brov2_description)/meshes/prop.dae"/>
+  <xacro:property name="prop_mesh_file" value="file://$(find brov2_description)/meshes/brov2_prop.dae"/>
   <!-- Copy Rexrov Thruster joint and link snippet -->
   <xacro:macro name="thruster_macro"
@@ -27,26 +27,26 @@
   </xacro:macro>
   <xacro:thruster_macro namespace="${namespace}" thruster_id="0">
-    <origin xyz="-0.890895 0.334385 0.528822" rpy="${0*d2r} ${-74.53*d2r} ${-53.21*d2r}"/>
+    <origin xyz="0.1489 0.0908 0.0647" rpy="${0*d2r} ${0*d2r} ${135*d2r}"/>
   </xacro:thruster_macro>
   <xacro:thruster_macro namespace="${namespace}" thruster_id="1">
-    <origin xyz="-0.890895 -0.334385 0.528822" rpy="${0*d2r} ${-74.53*d2r} ${53.21*d2r}"/>
+    <origin xyz="0.1489 -0.1029 0.0647" rpy="${0*d2r} ${0*d2r} ${225*d2r}"/>
   </xacro:thruster_macro>
   <xacro:thruster_macro namespace="${namespace}" thruster_id="2">
-    <origin xyz="0.890895 0.334385 0.528822" rpy="${0*d2r} ${-105.47*d2r} ${53.21*d2r}"/>
+    <origin xyz="-0.1526 0.0906 0.0647" rpy="${0*d2r} ${0*d2r} ${45*d2r}"/>
   </xacro:thruster_macro>
   <xacro:thruster_macro namespace="${namespace}" thruster_id="3">
-    <origin xyz="0.890895 -0.334385 0.528822" rpy="${0*d2r} ${-105.47*d2r} ${-53.21*d2r}"/>
+    <origin xyz="-0.1526 -0.1027 0.0647" rpy="${0*d2r} ${0*d2r} ${315*d2r}"/>
   </xacro:thruster_macro>
   <xacro:thruster_macro namespace="${namespace}" thruster_id="4">
-    <origin xyz="-0.412125 0.505415 0.129" rpy="${0*d2r} ${0*d2r} ${45*d2r}"/>
+    <origin xyz="0.1255 0.212 -0.0125" rpy="${0*d2r} ${-90*d2r} ${0*d2r}"/>
   </xacro:thruster_macro>
   <xacro:thruster_macro namespace="${namespace}" thruster_id="5">
-    <origin xyz="-0.412125 -0.505415 0.129" rpy="${0*d2r} ${0*d2r} ${-45*d2r}"/>
+    <origin xyz="0.1255 -0.2241 -0.0109" rpy="${0*d2r} ${-90*d2r} ${0*d2r}"/>
   </xacro:thruster_macro>
   <xacro:thruster_macro namespace="${namespace}" thruster_id="6">
-    <origin xyz="0.412125 0.505415 0.129" rpy="${0*d2r} ${0*d2r} ${135*d2r}"/>
+    <origin xyz="-0.1145 0.212 -0.0109" rpy="${0*d2r} ${-90*d2r} ${0*d2r}"/>
   </xacro:thruster_macro>
   <xacro:thruster_macro namespace="${namespace}" thruster_id="7">
-    <origin xyz="0.412125 -0.505415 0.129" rpy="${0*d2r} ${0*d2r} ${-135*d2r}"/>
+    <origin xyz="-0.1145 -0.2241 -0.0125" rpy="${0*d2r} ${-90*d2r} ${0*d2r}"/>
   </xacro:thruster_macro>
 </robot>

File: urdf/robots/brov2_description/urdf/brov2_base.xacro (robot description, xacro)
@@ -29,5 +29,5 @@
   <xacro:property name="namespace" value="brov2"/>
   <xacro:property name="visual_mesh_file" value="file://$(find brov2_description)/meshes/brov2.dae"/>
-  <xacro:property name="prop_mesh_file" value="file://$(find brov2_description)/meshes/prop.dae"/>
+  <xacro:property name="prop_mesh_file" value="file://$(find brov2_description)/meshes/brov2_prop.dae"/>
   <!-- Mass, see p.48 in Wu2018 -->
   <xacro:property name="mass" value="11.5"/>

File: urdf/robots/brov2_description/urdf/brov2_sensors.xacro (robot description, xacro)
@@ -15,20 +15,21 @@
 <!-- copy rexrov_sensors for now -->
   <!-- DVL  -->
-  <xacro:default_dvl_macro
+  <!-- <xacro:default_dvl_macro
     namespace="${namespace}"
     parent_link="${namespace}/base_link"
     inertial_reference_frame="${inertial_reference_frame}">
     <origin xyz="-1.4 0 -0.312" rpy="0 ${0.5*pi} 0"/>
-  </xacro:default_dvl_macro>
+  </xacro:default_dvl_macro> -->
   <!-- Magnetometer  -->
-  <xacro:default_magnetometer namespace="${namespace}" parent_link="${namespace}/base_link"/>
+  <!-- <xacro:default_magnetometer namespace="${namespace}" parent_link="${namespace}/base_link"/> -->
   <!-- RPT  -->
-  <xacro:default_rpt namespace="${namespace}" parent_link="${namespace}/base_link">
+  <!-- <xacro:default_rpt namespace="${namespace}" parent_link="${namespace}/base_link">
     <origin xyz="-1.32 0 0.8" rpy="0 0 0"/>
-  </xacro:default_rpt>
+  </xacro:default_rpt> -->
   <!-- Pressure  -->
-  <xacro:default_pressure_macro namespace="${namespace}" parent_link="${namespace}/base_link">
-    <origin xyz="-1.32 0.5 0.85" rpy="0 0 0"/>
-  </xacro:default_pressure_macro>
+  <!-- <xacro:default_pressure_macro namespace="${namespace}" parent_link="${namespace}/base_link"> -->
+    <!-- <origin xyz="-1.32 0.5 0.85" rpy="0 0 0"/> -->
+  <!-- </xacro:default_pressure_macro> -->
+<!--  -->
   <!-- IMU  -->
   <xacro:default_imu_macro
@@ -39,13 +40,13 @@
   </xacro:default_imu_macro>
   <!-- Mount a camera -->
-  <xacro:default_camera namespace="${namespace}" parent_link="${namespace}/base_link" suffix="">
+  <!-- <xacro:default_camera namespace="${namespace}" parent_link="${namespace}/base_link" suffix="">
     <origin xyz="1.15 0 0.4" rpy="0 0.6 0"/>
-  </xacro:default_camera>
-  <xacro:default_camera namespace="${namespace}" parent_link="${namespace}/base_link" suffix="right">
+  </xacro:default_camera> -->
+  <!-- <xacro:default_camera namespace="${namespace}" parent_link="${namespace}/base_link" suffix="right">
     <origin xyz="1.15 -0.63 0.4" rpy="0 0.6 0.4"/>
   </xacro:default_camera>
   <xacro:default_camera namespace="${namespace}" parent_link="${namespace}/base_link" suffix="left">
     <origin xyz="1.15 0.63 0.4" rpy="0 0.6 -0.4"/>
-  </xacro:default_camera>
+  </xacro:default_camera> -->
   <!-- Mount a Pose 3D sensor. -->
   <xacro:default_pose_3d_macro

Commit message: save point for ned

File: urdf/robots/brov2_description/urdf/brov2.gazebo.xacro (robot description, xacro)
@@ -18,5 +18,5 @@
     <xacro:property name="cob" value="0.0 0.0 0.0"/>
     <!-- overestimated cube based on brov2 dimensions https://bluerobotics.com/store/rov/bluerov2-upgrade-kits/brov2-heavy-retrofit/ -->
-    <xacro:property name="volume" value="0.0661"/>
+    <xacro:property name="volume" value="0.01142"/>
     <xacro:macro name="brov2_hydro_model" params="namespace">
         <link name="${namespace}/base_link">

File: urdf/robots/brov2_description/urdf/brov2.xacro (robot description, xacro)
@@ -15,5 +15,5 @@
   <xacro:arg name="debug" default="0"/>
   <xacro:arg name="namespace" default="brov2"/>
-  <xacro:arg name="inertial_reference_frame" default="world"/>
+  <xacro:arg name="inertial_reference_frame" default="world_ned"/>
   <!-- Include the ROV macro file -->
   <xacro:include filename="$(find brov2_description)/urdf/brov2_base.xacro"/>

File: urdf/robots/brov2_description/urdf/brov2_actuators.xacro (robot description, xacro)
@@ -26,5 +26,5 @@
     </xacro:thruster_module_first_order_basic_fcn_macro>
   </xacro:macro>
-  <xacro:thruster_macro namespace="${namespace}" thruster_id="0">
+  <!-- <xacro:thruster_macro namespace="${namespace}" thruster_id="0">
     <origin xyz="0.1489 0.0908 0.0647" rpy="${0*d2r} ${0*d2r} ${135*d2r}"/>
   </xacro:thruster_macro>
@@ -39,5 +39,5 @@
   </xacro:thruster_macro>
   <xacro:thruster_macro namespace="${namespace}" thruster_id="4">
-    <origin xyz="0.1255 0.212 -0.0125" rpy="${0*d2r} ${-90*d2r} ${0*d2r}"/>
+    <origin xyz="0.1255 0.212 0.0125" rpy="${0*d2r} ${-90*d2r} ${0*d2r}"/>
   </xacro:thruster_macro>
   <xacro:thruster_macro namespace="${namespace}" thruster_id="5">
@@ -49,4 +49,28 @@
   <xacro:thruster_macro namespace="${namespace}" thruster_id="7">
     <origin xyz="-0.1145 -0.2241 -0.0125" rpy="${0*d2r} ${-90*d2r} ${0*d2r}"/>
+  </xacro:thruster_macro> -->
+  <xacro:thruster_macro namespace="${namespace}" thruster_id="0">
+    <origin xyz="0.1489 0.0908 0.06" rpy="${0*d2r} ${0*d2r} ${225*d2r}"/>
+  </xacro:thruster_macro>
+  <xacro:thruster_macro namespace="${namespace}" thruster_id="1">
+    <origin xyz="0.1489 -0.09 0.06" rpy="${0*d2r} ${0*d2r} ${135*d2r}"/>
+  </xacro:thruster_macro>
+  <xacro:thruster_macro namespace="${namespace}" thruster_id="2">
+    <origin xyz="-0.1489 0.0906 0.06" rpy="${0*d2r} ${0*d2r} ${-45*d2r}"/>
+  </xacro:thruster_macro>
+  <xacro:thruster_macro namespace="${namespace}" thruster_id="3">
+    <origin xyz="-0.1489 -0.0906 0.06" rpy="${0*d2r} ${0*d2r} ${45*d2r}"/>
+  </xacro:thruster_macro>
+  <xacro:thruster_macro namespace="${namespace}" thruster_id="4">
+    <origin xyz="0.1255 0.212 -0.0125" rpy="${0*d2r} ${-90*d2r} ${0*d2r}"/>
+  </xacro:thruster_macro>
+  <xacro:thruster_macro namespace="${namespace}" thruster_id="5">
+    <origin xyz="0.1255 -0.212 -0.0125" rpy="${0*d2r} ${-90*d2r} ${0*d2r}"/>
+  </xacro:thruster_macro>
+  <xacro:thruster_macro namespace="${namespace}" thruster_id="6">
+    <origin xyz="-0.1255 0.212 -0.0125" rpy="${0*d2r} ${-90*d2r} ${0*d2r}"/>
+  </xacro:thruster_macro>
+  <xacro:thruster_macro namespace="${namespace}" thruster_id="7">
+    <origin xyz="-0.1255 -0.212 -0.0125" rpy="${0*d2r} ${-90*d2r} ${0*d2r}"/>
   </xacro:thruster_macro>
 </robot>

Commit message: changed brov to z-up

File: urdf/robots/brov2_description/urdf/brov2.gazebo.xacro (robot description, xacro)
@@ -16,10 +16,10 @@
     Center of buoyancy according to Table 5.1 p. 48 in Wu2018.
     -->
-    <xacro:property name="cob" value="0.0 0.0 0.0"/>
+    <xacro:property name="cob" value="0.0 0.0 0.2"/>
     <!-- overestimated cube based on brov2 dimensions https://bluerobotics.com/store/rov/bluerov2-upgrade-kits/brov2-heavy-retrofit/ -->
     <xacro:property name="volume" value="0.0661"/>
     <xacro:macro name="brov2_hydro_model" params="namespace">
         <link name="${namespace}/base_link">
-            <neutrally_buoyant>0</neutrally_buoyant>
+            <neutrally_buoyant>1</neutrally_buoyant>
             <volume>${volume}</volume>
             <box>
@@ -33,10 +33,10 @@
                 <!-- Added mass: see p.28 Table 5.2 p. 48 in Wu2018 -->
                 <added_mass>
-                    -5.5   0.0  0.0    0.0   0.0   0.0
-                    0.0   -12.7 0.0    0.0   0.0   0.0
-                    0.0   0.0  -14.57  0.0   0.0   0.0
-                    0.0   0.0  0.0    -0.12  0.0   0.0
-                    0.0   0.0  0.0     0.0  -0.12  0.0
-                    0.0   0.0  0.0     0.0   0.0  -0.12
+                    5.5   0.0  0.0    0.0   0.0   0.0
+                    0.0   12.7 0.0    0.0   0.0   0.0
+                    0.0   0.0  14.57  0.0   0.0   0.0
+                    0.0   0.0  0.0    0.12  0.0   0.0
+                    0.0   0.0  0.0    0.0   0.12  0.0
+                    0.0   0.0  0.0    0.0   0.0   0.12
                 </added_mass>
                 <!-- Linear Damping: see Table 5.3 p. 48 in Wu2018 -->
@@ -59,3 +59,9 @@
                     0.0   0.0  0.0    0.0   0.0   0.12
                 </added_mass> -->
+                    <!-- -5.5   0.0  0.0    0.0   0.0   0.0
+                    0.0   -12.7 0.0    0.0   0.0   0.0
+                    0.0   0.0  -14.57  0.0   0.0   0.0
+                    0.0   0.0  0.0    -0.12  0.0   0.0
+                    0.0   0.0  0.0     0.0  -0.12  0.0
+                    0.0   0.0  0.0     0.0   0.0  -0.12 -->
 </robot>

File: urdf/robots/brov2_description/urdf/brov2_actuators.xacro (robot description, xacro)
@@ -22,31 +22,55 @@
       mesh_filename="${prop_mesh_file}"
       dyn_time_constant="0.05"
-      rotor_constant="0.00031">
+      rotor_constant="0.0003">
       <xacro:insert_block name="origin"/>
     </xacro:thruster_module_first_order_basic_fcn_macro>
   </xacro:macro>
   <xacro:thruster_macro namespace="${namespace}" thruster_id="0">
-    <origin xyz="0.1489 0.0908 0.0647" rpy="${0*d2r} ${0*d2r} ${135*d2r}"/>
+    <origin xyz="0.156 -0.111 -0.085" rpy="${0*d2r} ${0*d2r} ${45*d2r}"/>
   </xacro:thruster_macro>
   <xacro:thruster_macro namespace="${namespace}" thruster_id="1">
-    <origin xyz="0.1489 -0.1029 0.0647" rpy="${0*d2r} ${0*d2r} ${225*d2r}"/>
+    <origin xyz="0.156 0.111 -0.085" rpy="${0*d2r} ${0*d2r} ${315*d2r}"/>
   </xacro:thruster_macro>
   <xacro:thruster_macro namespace="${namespace}" thruster_id="2">
-    <origin xyz="-0.1526 0.0906 0.0647" rpy="${0*d2r} ${0*d2r} ${45*d2r}"/>
+    <origin xyz="-0.156 -0.111 -0.085" rpy="${0*d2r} ${0*d2r} ${135*d2r}"/>
   </xacro:thruster_macro>
   <xacro:thruster_macro namespace="${namespace}" thruster_id="3">
-    <origin xyz="-0.1526 -0.1027 0.0647" rpy="${0*d2r} ${0*d2r} ${315*d2r}"/>
+    <origin xyz="-0.156 0.111 -0.085" rpy="${0*d2r} ${0*d2r} ${225*d2r}"/>
   </xacro:thruster_macro>
   <xacro:thruster_macro namespace="${namespace}" thruster_id="4">
-    <origin xyz="0.1255 0.212 -0.0125" rpy="${0*d2r} ${-90*d2r} ${0*d2r}"/>
+    <origin xyz="0.120 -0.218 0.0" rpy="${0*d2r} ${90*d2r} ${0*d2r}"/>
   </xacro:thruster_macro>
   <xacro:thruster_macro namespace="${namespace}" thruster_id="5">
-    <origin xyz="0.1255 -0.2241 -0.0109" rpy="${0*d2r} ${-90*d2r} ${0*d2r}"/>
+    <origin xyz="0.120 0.218 0.0" rpy="${0*d2r} ${90*d2r} ${0*d2r}"/>
   </xacro:thruster_macro>
   <xacro:thruster_macro namespace="${namespace}" thruster_id="6">
-    <origin xyz="-0.1145 0.212 -0.0109" rpy="${0*d2r} ${-90*d2r} ${0*d2r}"/>
+    <origin xyz="-0.120 -0.218 0.0" rpy="${0*d2r} ${90*d2r} ${0*d2r}"/>
   </xacro:thruster_macro>
   <xacro:thruster_macro namespace="${namespace}" thruster_id="7">
-    <origin xyz="-0.1145 -0.2241 -0.0125" rpy="${0*d2r} ${-90*d2r} ${0*d2r}"/>
+    <origin xyz="-0.120 0.218 0.0" rpy="${0*d2r} ${90*d2r} ${0*d2r}"/>
   </xacro:thruster_macro>
+  <!-- <xacro:thruster_macro namespace="${namespace}" thruster_id="0">
+    <origin xyz="0.1489 0.0908 -0.0647" rpy="${0*d2r} ${0*d2r} ${135*d2r}"/>
+  </xacro:thruster_macro>
+  <xacro:thruster_macro namespace="${namespace}" thruster_id="1">
+    <origin xyz="0.1489 -0.1029 -0.0647" rpy="${0*d2r} ${0*d2r} ${225*d2r}"/>
+  </xacro:thruster_macro>
+  <xacro:thruster_macro namespace="${namespace}" thruster_id="2">
+    <origin xyz="-0.1526 0.0906 -0.0647" rpy="${0*d2r} ${0*d2r} ${45*d2r}"/>
+  </xacro:thruster_macro>
+  <xacro:thruster_macro namespace="${namespace}" thruster_id="3">
+    <origin xyz="-0.1526 -0.1027 -0.0647" rpy="${0*d2r} ${0*d2r} ${315*d2r}"/>
+  </xacro:thruster_macro>
+  <xacro:thruster_macro namespace="${namespace}" thruster_id="4">
+    <origin xyz="0.1255 0.212 0.0125" rpy="${0*d2r} ${-90*d2r} ${0*d2r}"/>
+  </xacro:thruster_macro>
+  <xacro:thruster_macro namespace="${namespace}" thruster_id="5">
+    <origin xyz="0.1255 -0.2241 0.0125" rpy="${0*d2r} ${-90*d2r} ${0*d2r}"/>
+  </xacro:thruster_macro>
+  <xacro:thruster_macro namespace="${namespace}" thruster_id="6">
+    <origin xyz="-0.1145 0.212 0.0125" rpy="${0*d2r} ${-90*d2r} ${0*d2r}"/>
+  </xacro:thruster_macro>
+  <xacro:thruster_macro namespace="${namespace}" thruster_id="7">
+    <origin xyz="-0.1145 -0.2241 0.0125" rpy="${0*d2r} ${-90*d2r} ${0*d2r}"/>
+  </xacro:thruster_macro> -->
 </robot>
